File: software/test_data/circuit/circuit.sch (KiCad schematic (older format))
At the start: 18 parts

Commit message: update circuit to include separate power control for DC motor
Parts:
- removed J? (x3): Conn_01x04_Male, symbol Connector:Conn_01x04_Male
- added D? (x2): LED, symbol Device:LED
- added K?: UMS05-1A80-75L, Relay_THT:Relay_StandexMeder_UMS, symbol Relay:UMS05-1A80-75L
- added M?: Motor_DC, symbol Motor:Motor_DC
- added M? (x3): Stepper_Motor_bipolar, symbol Motor:Stepper_Motor_bipolar
- added Q?: Q_NMOS_DGS, symbol Device:Q_NMOS_DGS
- added Q?: NMOS_GSD_30V, footprints:SOT-23F, symbol formula:NMOS_GSD_30V
- added Q?: Q_PMOS_DGS, symbol Device:Q_PMOS_DGS
- added R?: R_1k, symbol Device:R
- added R?: R_200, symbol Device:R
Connections:
- net labels added: 12V_Dremel
- wire segments 117 -> 160
- no-connect marks 14 -> 15

Commit message: update to make axis change circuit
Parts:
- added D? (x2): LED, symbol Device:LED
- added R?: R_10k, symbol Device:R
- added R? (x2): R_200, symbol Device:R
Connections:
- net labels added: AxisChange, LED0, LED1
- wire segments 160 -> 175
- no-connect marks 15 -> 11

Commit message: updated schematic with nfet driving the brushed motor
Parts:
- added Q?: Q_NMOS_DGS, symbol Device:Q_NMOS_DGS
Connections:
- net labels added: PWM_Motor
- wire segments 175 -> 178
- no-connect marks 11 -> 10
Changed lines of the file:
@@
 NoConn ~ 7150 3550
 NoConn ~ 7150 3650
-NoConn ~ 6150 2750
 $Comp
 L Device:R_POT RV?
@@
 L Relay:UMS05-1A80-75L K?
 U 1 1 5C076FB4
-P 6600 5150
-F 0 "K?" H 6880 5196 50  0000 L CNN
-F 1 "UMS05-1A80-75L" H 6880 5105 50  0000 L CNN
-F 2 "Relay_THT:Relay_StandexMeder_UMS" H 6900 5100 50  0001 L CNN
-F 3 "https://standexelectronics.com/de/produkte/ums-reed-relais/" H 6600 5150 50  0001 C CNN
-	1    6600 5150
+P 6600 5000
+F 0 "K?" H 6880 5046 50  0000 L CNN
+F 1 "UMS05-1A80-75L" H 6880 4955 50  0000 L CNN
+F 2 "Relay_THT:Relay_StandexMeder_UMS" H 6900 4950 50  0001 L CNN
+F 3 "https://standexelectronics.com/de/produkte/ums-reed-relais/" H 6600 5000 50  0001 C CNN
+	1    6600 5000
 	1    0    0    -1
 $EndComp
@@
 L Device:Q_NMOS_DGS Q?
 U 1 1 5C07726E
-P 6300 5800
-F 0 "Q?" H 6505 5846 50  0000 L CNN
-F 1 "Q_NMOS_DGS" H 6505 5755 50  0000 L CNN
-F 2 "" H 6500 5900 50  0001 C CNN
-F 3 "~" H 6300 5800 50  0001 C CNN
-	1    6300 5800
-	1    0    0    -1
-$EndComp
-Wire Wire Line
-	6400 5450 6400 5600
-Wire Wire Line
-	6400 6000 6400 6100
+P 6300 5650
+F 0 "Q?" H 6505 5696 50  0000 L CNN
+F 1 "Q_NMOS_DGS" H 6505 5605 50  0000 L CNN
+F 2 "" H 6500 5750 50  0001 C CNN
+F 3 "~" H 6300 5650 50  0001 C CNN
+	1    6300 5650
+	1    0    0    -1
+$EndComp
+Wire Wire Line
+	6400 5300 6400 5450
+Wire Wire Line
+	6400 5850 6400 5950
 $Comp
 L power:GND #PWR?
 U 1 1 5C07F8CB
-P 6400 6100
-F 0 "#PWR?" H 6400 5850 50  0001 C CNN
-F 1 "GND" H 6405 5927 50  0000 C CNN
-F 2 "" H 6400 6100 50  0001 C CNN
-F 3 "" H 6400 6100 50  0001 C CNN
-	1    6400 6100
+P 6400 5950
+F 0 "#PWR?" H 6400 5700 50  0001 C CNN
+F 1 "GND" H 6500 5850 50  0000 C CNN
+F 2 "" H 6400 5950 50  0001 C CNN
+F 3 "" H 6400 5950 50  0001 C CNN
+	1    6400 5950
 	1    0    0    -1
 $EndComp
@@
 L Motor:Motor_DC M?
 U 1 1 5C07FC71
-P 7400 5750
-F 0 "M?" H 7558 5746 50  0000 L CNN
-F 1 "Motor_DC" H 7558 5655 50  0000 L CNN
-F 2 "" H 7400 5660 50  0001 C CNN
-F 3 "~" H 7400 5660 50  0001 C CNN
-	1    7400 5750
-	1    0    0    -1
-$EndComp
-Wire Wire Line
-	6800 5450 6800 5550
-Wire Wire Line
-	6800 5550 7400 5550
-Wire Wire Line
-	7400 6050 7400 6100
-$Comp
-L power:GND #PWR?
-U 1 1 5C0887E8
-P 7400 6100
-F 0 "#PWR?" H 7400 5850 50  0001 C CNN
-F 1 "GND" H 7405 5927 50  0000 C CNN
-F 2 "" H 7400 6100 50  0001 C CNN
-F 3 "" H 7400 6100 50  0001 C CNN
-	1    7400 6100
-	1    0    0    -1
-$EndComp
-Wire Wire Line
-	6800 4850 6800 4600
-Wire Wire Line
-	6400 4850 6400 4700
+P 7400 5600
+F 0 "M?" H 7558 5596 50  0000 L CNN
+F 1 "Motor_DC" H 7558 5505 50  0000 L CNN
+F 2 "" H 7400 5510 50  0001 C CNN
+F 3 "~" H 7400 5510 50  0001 C CNN
+	1    7400 5600
+	1    0    0    -1
+$EndComp
+Wire Wire Line
+	6800 5300 6800 5400
+Wire Wire Line
+	6800 5400 7400 5400
+Wire Wire Line
+	7400 5900 7400 6150
+Wire Wire Line
+	6800 4700 6800 4450
+Wire Wire Line
+	6400 4700 6400 4550
 $Comp
 L power:+12V #PWR?
 U 1 1 5C091656
-P 6400 4700
-F 0 "#PWR?" H 6400 4550 50  0001 C CNN
-F 1 "+12V" H 6415 4873 50  0000 C CNN
-F 2 "" H 6400 4700 50  0001 C CNN
-F 3 "" H 6400 4700 50  0001 C CNN
-	1    6400 4700
-	1    0    0    -1
-$EndComp
-Text Label 6800 4600 0    50   ~ 0
+P 6400 4550
+F 0 "#PWR?" H 6400 4400 50  0001 C CNN
+F 1 "+12V" H 6415 4723 50  0000 C CNN
+F 2 "" H 6400 4550 50  0001 C CNN
+F 3 "" H 6400 4550 50  0001 C CNN
+	1    6400 4550
+	1    0    0    -1
+$EndComp
+Text Label 6800 4450 0    50   ~ 0
 12V_Dremel
 $Comp
 L formula:NMOS_GSD_30V Q?
 U 1 1 5C0A89C4
-P 5800 6050
-F 0 "Q?" H 6006 6096 50  0000 L CNN
-F 1 "NMOS_GSD_30V" H 6006 6005 50  0000 L CNN
-F 2 "footprints:SOT-23F" H 6000 6150 50  0001 C CNN
-F 3 "https://www.digikey.com/products/en?keywords=SSM3K333RLFCT-ND" H 6000 6100 50  0001 C CNN
-F 4 "Digi-Key" H 5800 6050 60  0001 C CNN "MFN"
-F 5 "SSM3K333RLFCT-ND" H 5800 6050 60  0001 C CNN "MPN"
-F 6 "Value" H 5800 6050 60  0001 C CNN "Package"
-F 7 "https://www.digikey.com/products/en?keywords=SSM3K333RLFCT-ND" H 6400 6500 60  0001 C CNN "PurchasingLink"
-	1    5800 6050
+P 5800 5900
+F 0 "Q?" H 6006 5946 50  0000 L CNN
+F 1 "NMOS_GSD_30V" H 6006 5855 50  0000 L CNN
+F 2 "footprints:SOT-23F" H 6000 6000 50  0001 C CNN
+F 3 "https://www.digikey.com/products/en?keywords=SSM3K333RLFCT-ND" H 6000 5950 50  0001 C CNN
+F 4 "Digi-Key" H 5800 5900 60  0001 C CNN "MFN"
+F 5 "SSM3K333RLFCT-ND" H 5800 5900 60  0001 C CNN "MPN"
+F 6 "Value" H 5800 5900 60  0001 C CNN "Package"
+F 7 "https://www.digikey.com/products/en?keywords=SSM3K333RLFCT-ND" H 6400 6350 60  0001 C CNN "PurchasingLink"
+	1    5800 5900
 	1    0    0    -1
 $EndComp
@@
 L power:GND #PWR?
 U 1 1 5C0AD349
-P 5900 6350
-F 0 "#PWR?" H 5900 6100 50  0001 C CNN
-F 1 "GND" H 5905 6177 50  0000 C CNN
-F 2 "" H 5900 6350 50  0001 C CNN
-F 3 "" H 5900 6350 50  0001 C CNN
-	1    5900 6350
-	1    0    0    -1
-$EndComp
-Wire Wire Line
-	5900 6250 5900 6350
+P 5900 6200
+F 0 "#PWR?" H 5900 5950 50  0001 C CNN
+F 1 "GND" H 6000 6100 50  0000 C CNN
+F 2 "" H 5900 6200 50  0001 C CNN
+F 3 "" H 5900 6200 50  0001 C CNN
+	1    5900 6200
+	1    0    0    -1
+$EndComp
+Wire Wire Line
+	5900 6100 5900 6200
 $Comp
 L Device:Q_PMOS_DGS Q?
 U 1 1 5C0B261F
-P 5800 5550
-F 0 "Q?" H 6006 5504 50  0000 L CNN
-F 1 "Q_PMOS_DGS" H 6006 5595 50  0000 L CNN
-F 2 "" H 6000 5650 50  0001 C CNN
-F 3 "~" H 5800 5550 50  0001 C CNN
-	1    5800 5550
+P 5800 5400
+F 0 "Q?" H 6006 5354 50  0000 L CNN
+F 1 "Q_PMOS_DGS" H 6006 5445 50  0000 L CNN
+F 2 "" H 6000 5500 50  0001 C CNN
+F 3 "~" H 5800 5400 50  0001 C CNN
+	1    5800 5400
 	1    0    0    1
 $EndComp
 Wire Wire Line
-	5200 4300 5200 5550
-Wire Wire Line
-	5600 6050 5200 6050
-Connection ~ 5200 6050
-Wire Wire Line
-	5200 6050 5200 6150
-Wire Wire Line
-	5600 5550 5200 5550
-Connection ~ 5200 5550
-Wire Wire Line
-	5200 5550 5200 6050
-Wire Wire Line
-	5900 5750 5900 5800
-Wire Wire Line
-	5900 5800 6100 5800
-Wire Wire Line
-	5900 5800 5900 5850
-Connection ~ 5900 5800
-Wire Wire Line
-	5900 4700 5900 5350
+	5200 4300 5200 5400
+Wire Wire Line
+	5600 5900 5200 5900
+Connection ~ 5200 5900
+Wire Wire Line
+	5200 5900 5200 6150
+Wire Wire Line
+	5600 5400 5200 5400
+Connection ~ 5200 5400
+Wire Wire Line
+	5200 5400 5200 5900
+Wire Wire Line
+	5900 5600 5900 5650
+Wire Wire Line
+	5900 5650 6100 5650
+Wire Wire Line
+	5900 5650 5900 5700
+Connection ~ 5900 5650
+Wire Wire Line
+	5900 4550 5900 5200
 $Comp
 L power:+5V #PWR?
 U 1 1 5C0E252A
-P 5900 4700
-F 0 "#PWR?" H 5900 4550 50  0001 C CNN
-F 1 "+5V" H 5915 4873 50  0000 C CNN
-F 2 "" H 5900 4700 50  0001 C CNN
-F 3 "" H 5900 4700 50  0001 C CNN
-	1    5900 4700
+P 5900 4550
+F 0 "#PWR?" H 5900 4400 50  0001 C CNN
+F 1 "+5V" H 5915 4723 50  0000 C CNN
+F 2 "" H 5900 4550 50  0001 C CNN
+F 3 "" H 5900 4550 50  0001 C CNN
+	1    5900 4550
 	1    0    0    -1
 $EndComp
@@
 	1    0    0    -1
 $EndComp
+$Comp
+L Device:Q_NMOS_DGS Q?
+U 1 1 5C071AB7
+P 7300 6350
+F 0 "Q?" H 7505 6396 50  0000 L CNN
+F 1 "Q_NMOS_DGS" H 7505 6305 50  0000 L CNN
+F 2 "" H 7500 6450 50  0001 C CNN
+F 3 "~" H 7300 6350 50  0001 C CNN
+	1    7300 6350
+	1    0    0    -1
+$EndComp
+$Comp
+L power:GND #PWR?
+U 1 1 5C071B2E
+P 7400 6550
+F 0 "#PWR?" H 7400 6300 50  0001 C CNN
+F 1 "GND" H 7405 6377 50  0000 C CNN
+F 2 "" H 7400 6550 50  0001 C CNN
+F 3 "" H 7400 6550 50  0001 C CNN
+	1    7400 6550
+	1    0    0    -1
+$EndComp
+Wire Wire Line
+	7100 6350 5550 6350
+Wire Wire Line
+	5550 6350 5550 2750
+Wire Wire Line
+	5550 2750 6150 2750
+Text Label 5750 2750 0    50   ~ 0
+PWM_Motor
 $EndSCHEMATC

Commit message: adding circuit images
Parts:
- removed Q?: NMOS_GSD_30V, footprints:SOT-23F, symbol formula:NMOS_GSD_30V
- removed Q?: Q_PMOS_DGS, symbol Device:Q_PMOS_DGS
- added R? (x2): R, symbol Device:R
- added U?: 74HC04, symbol 74xx:74HC04
Connections:
- wire segments 178 -> 175
Changed lines of the file:
@@
 L Device:Q_NMOS_DGS Q?
 U 1 1 5C07726E
-P 6300 5650
-F 0 "Q?" H 6505 5696 50  0000 L CNN
-F 1 "Q_NMOS_DGS" H 6505 5605 50  0000 L CNN
-F 2 "" H 6500 5750 50  0001 C CNN
-F 3 "~" H 6300 5650 50  0001 C CNN
-	1    6300 5650
-	1    0    0    -1
-$EndComp
-Wire Wire Line
-	6400 5300 6400 5450
-Wire Wire Line
-	6400 5850 6400 5950
+P 6550 5900
+F 0 "Q?" H 6755 5946 50  0000 L CNN
+F 1 "Q_NMOS_DGS" H 6755 5855 50  0000 L CNN
+F 2 "" H 6750 6000 50  0001 C CNN
+F 3 "~" H 6550 5900 50  0001 C CNN
+	1    6550 5900
+	1    0    0    -1
+$EndComp
+Wire Wire Line
+	6650 6100 6650 6200
 $Comp
 L power:GND #PWR?
 U 1 1 5C07F8CB
-P 6400 5950
-F 0 "#PWR?" H 6400 5700 50  0001 C CNN
-F 1 "GND" H 6500 5850 50  0000 C CNN
-F 2 "" H 6400 5950 50  0001 C CNN
-F 3 "" H 6400 5950 50  0001 C CNN
-	1    6400 5950
+P 6650 6200
+F 0 "#PWR?" H 6650 5950 50  0001 C CNN
+F 1 "GND" H 6750 6100 50  0000 C CNN
+F 2 "" H 6650 6200 50  0001 C CNN
+F 3 "" H 6650 6200 50  0001 C CNN
+	1    6650 6200
 	1    0    0    -1
 $EndComp
@@
 Text Label 6800 4450 0    50   ~ 0
 12V_Dremel
-$Comp
-L formula:NMOS_GSD_30V Q?
-U 1 1 5C0A89C4
-P 5800 5900
-F 0 "Q?" H 6006 5946 50  0000 L CNN
-F 1 "NMOS_GSD_30V" H 6006 5855 50  0000 L CNN
-F 2 "footprints:SOT-23F" H 6000 6000 50  0001 C CNN
-F 3 "https://www.digikey.com/products/en?keywords=SSM3K333RLFCT-ND" H 6000 5950 50  0001 C CNN
-F 4 "Digi-Key" H 5800 5900 60  0001 C CNN "MFN"
-F 5 "SSM3K333RLFCT-ND" H 5800 5900 60  0001 C CNN "MPN"
-F 6 "Value" H 5800 5900 60  0001 C CNN "Package"
-F 7 "https://www.digikey.com/products/en?keywords=SSM3K333RLFCT-ND" H 6400 6350 60  0001 C CNN "PurchasingLink"
-	1    5800 5900
-	1    0    0    -1
-$EndComp
-$Comp
-L power:GND #PWR?
-U 1 1 5C0AD349
-P 5900 6200
-F 0 "#PWR?" H 5900 5950 50  0001 C CNN
-F 1 "GND" H 6000 6100 50  0000 C CNN
-F 2 "" H 5900 6200 50  0001 C CNN
-F 3 "" H 5900 6200 50  0001 C CNN
-	1    5900 6200
-	1    0    0    -1
-$EndComp
-Wire Wire Line
-	5900 6100 5900 6200
-$Comp
-L Device:Q_PMOS_DGS Q?
-U 1 1 5C0B261F
-P 5800 5400
-F 0 "Q?" H 6006 5354 50  0000 L CNN
-F 1 "Q_PMOS_DGS" H 6006 5445 50  0000 L CNN
-F 2 "" H 6000 5500 50  0001 C CNN
-F 3 "~" H 5800 5400 50  0001 C CNN
-	1    5800 5400
-	1    0    0    1
-$EndComp
-Wire Wire Line
-	5200 4300 5200 5400
 Wire Wire Line
 	5600 5900 5200 5900
@@
 Wire Wire Line
 	5200 5900 5200 6150
-Wire Wire Line
-	5600 5400 5200 5400
-Connection ~ 5200 5400
-Wire Wire Line
-	5200 5400 5200 5900
-Wire Wire Line
-	5900 5600 5900 5650
-Wire Wire Line
-	5900 5650 6100 5650
-Wire Wire Line
-	5900 5650 5900 5700
-Connection ~ 5900 5650
-Wire Wire Line
-	5900 4550 5900 5200
-$Comp
-L power:+5V #PWR?
-U 1 1 5C0E252A
-P 5900 4550
-F 0 "#PWR?" H 5900 4400 50  0001 C CNN
-F 1 "+5V" H 5915 4723 50  0000 C CNN
-F 2 "" H 5900 4550 50  0001 C CNN
-F 3 "" H 5900 4550 50  0001 C CNN
-	1    5900 4550
-	1    0    0    -1
-$EndComp
 $Comp
 L Motor:Stepper_Motor_bipolar M?
@@
 $EndComp
 Wire Wire Line
-	7100 6350 5550 6350
+	7100 6350 6450 6350
 Wire Wire Line
 	5550 6350 5550 2750
@@
 Text Label 5750 2750 0    50   ~ 0
 PWM_Motor
+$Comp
+L 74xx:74HC04 U?
+U 1 1 5C075E91
+P 5900 5900
+F 0 "U?" H 5900 6217 50  0000 C CNN
+F 1 "74HC04" H 5900 6126 50  0000 C CNN
+F 2 "" H 5900 5900 50  0001 C CNN
+F 3 "http://www.nxp.com/documents/data_sheet/74HC_HCT04.pdf" H 5900 5900 50  0001 C CNN
+	1    5900 5900
+	1    0    0    -1
+$EndComp
+Wire Wire Line
+	5200 4300 5200 5900
+Wire Wire Line
+	6200 5900 6250 5900
+Wire Wire Line
+	6400 5700 6650 5700
+Wire Wire Line
+	6400 5300 6400 5700
+$Comp
+L Device:R R?
+U 1 1 5C098443
+P 6250 6050
+F 0 "R?" H 6320 6096 50  0000 L CNN
+F 1 "R" H 6320 6005 50  0000 L CNN
+F 2 "" V 6180 6050 50  0001 C CNN
+F 3 "~" H 6250 6050 50  0001 C CNN
+	1    6250 6050
+	1    0    0    -1
+$EndComp
+Connection ~ 6250 5900
+Wire Wire Line
+	6250 5900 6350 5900
+$Comp
+L power:GND #PWR?
+U 1 1 5C098557
+P 6250 6200
+F 0 "#PWR?" H 6250 5950 50  0001 C CNN
+F 1 "GND" H 6255 6027 50  0000 C CNN
+F 2 "" H 6250 6200 50  0001 C CNN
+F 3 "" H 6250 6200 50  0001 C CNN
+	1    6250 6200
+	1    0    0    -1
+$EndComp
+$Comp
+L Device:R R?
+U 1 1 5C0985F8
+P 6450 6500
+F 0 "R?" H 6520 6546 50  0000 L CNN
+F 1 "R" H 6520 6455 50  0000 L CNN
+F 2 "" V 6380 6500 50  0001 C CNN
+F 3 "~" H 6450 6500 50  0001 C CNN
+	1    6450 6500
+	1    0    0    -1
+$EndComp
+Connection ~ 6450 6350
+Wire Wire Line
+	6450 6350 5550 6350
+$Comp
+L power:GND #PWR?
+U 1 1 5C0986A4
+P 6450 6650
+F 0 "#PWR?" H 6450 6400 50  0001 C CNN
+F 1 "GND" H 6455 6477 50  0000 C CNN
+F 2 "" H 6450 6650 50  0001 C CNN
+F 3 "" H 6450 6650 50  0001 C CNN
+	1    6450 6650
+	1    0    0    -1
+$EndComp
 $EndSCHEMATC

Commit message: limit switch code; update schematic; website wit fix
Parts:
- added C?: C, symbol Device:C
- added R? (x2): R, symbol Device:R
- added SW? (x4): SW_Push, symbol Switch:SW_Push
Connections:
- net labels added: LimitSW
- wire segments 175 -> 197
- no-connect marks 10 -> 9
Other:
- moved on the sheet: U?A
